File: pcb/vfd-tool/vfd-tool.kicad_sch (KiCad schematic)
At the start: 163 parts, among them J1 Micro_SD_Card, J2 Conn_ARM_SWD_TagConnect_TC203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, J3 Conn_02x15_Odd_Even, J4 Raspberry_Pi_2_3, J5 USB_C_Receptacle_USB2.0, J6 Conn_02x15_Odd_Even, J7 Conn_02x08_Odd_Even, SW1 SW_Push, SW2 SW_Push, U1 RP2040, U10 TPS54331DR, U11 PCF85263AT, U2 W25Q32JVSS, U3 TPS562200, U4 TPS562200, U5 FUSB302BMPX, U6 BQ24075RGT, U7 MAX17048G_T10, U8 USB2514B_M2, U9 SRV05-4, Y1 24MHz, Y2 32.768kHz, Y3 24MHz

Commit message: USB + PD sections kinda done, started on battery charging
Parts:
- added J4: Conn_01x10, 5034801000:MOLEX_5034801000, symbol Connector_Generic:Conn_01x10
- added J9: Conn_01x02_Socket, Connector_JST:JST_PH_B2B-PH-SM4-TB_1x02-1MP_P2.00mm_Vertical, symbol Connector:Conn_01x02_Socket
- added TP1: VSYS, TestPoint:TestPoint_Pad_D3.0mm, symbol Connector:TestPoint
- added TP2: GND, TestPoint:TestPoint_Pad_D3.0mm, symbol Connector:TestPoint
- renumbered C36 to C10, C4 to C11, C39 to C12, C33 to C13, C40 to C14, C5 to C15, C32 to C16, C6 to C17, C7 to C18, C26 to C19, C8 to C20, C9 to C21, C10 to C22, C11 to C23, C12 to C24, C45 to C25, C60 to C26, C61 to C27, C46 to C28, C43 to C29, C38 to C3, C15 to C30, C59 to C31, C44 to C32, C47 to C33, C58 to C34, C48 to C35, C13 to C36, C14 to C37, C27 to C38, C49 to C39, C34 to C4, C16 to C40, C21 to C41, C50 to C42, C17 to C43, C22 to C44, C51 to C45, C52 to C46, C53 to C47, C28 to C48, C18 to C49, C35 to C5, C23 to C50, C54 to C51, C29 to C52, C19 to C53, C24 to C54, C31 to C57, C20 to C58, C25 to C59, C41 to C6, C57 to C60, C30 to C61, C37 to C7, C3 to C8, C42 to C9, D13 to D10, D8 to D11, D9 to D12, D10 to D13, D15 to D14, D3 to D2, D4 to D3, D5 to D4, D11 to D5, D2 to D6, D14 to D7, D12 to D8, D6 to D9, J2 to J1, J5 to J2, J1 to J3, J4 to J5, J3 to J6, J6 to J7, J7 to J8, R46 to R1, R13 to R10, R14 to R11, R15 to R12, R16 to R13, R40 to R14, R47 to R15, R57 to R16, R39 to R17, R23 to R18, R36 to R19, R11 to R2, R24 to R20, R41 to R21, R42 to R22, R43 to R23, R44 to R24, R50 to R25, R6 to R26, R49 to R27, R7 to R28, R48 to R29, R12 to R3, R8 to R30, R9 to R31, R54 to R32, R10 to R33, R55 to R34, R4 to R35, R5 to R36, R56 to R37, R25 to R38, R26 to R39, R45 to R4, R27 to R40, R28 to R41, R29 to R42, R17 to R43, R20 to R44, R32 to R45, R34 to R46, R35 to R47, R33 to R48, R51 to R49, R1 to R5, R30 to R50, R31 to R51, R18 to R52, R19 to R53, R21 to R54, R22 to R55, R52 to R56, R53 to R57, R2 to R6, R38 to R7, R3 to R8, R37 to R9, TP1 to TP3, TP2 to TP4, U6 to U11, U8 to U2, U9 to U3, U5 to U4, U11 to U5, U2 to U6, U3 to U7, U4 to U8, U7 to U9, Y3 to Y2, Y2 to Y3
Connections:
- net B+: now also J9.2 (Pin_2)
- net CC1: now also U3.4 (IO3)
- net CC2: now also U3.6 (IO4)
- net GND: now also BT1.N (-), J7.26 (Pin_26), J7.28 (Pin_28), J8.1 (Pin_1), J8.2 (Pin_2), J8.3 (Pin_3), J8.4 (Pin_4), J9.1 (Pin_1), TP2.1; no longer BT1.2 (-)
- net RPI0_GPIO4: no longer J5.7 (GCLK0/GPIO4)
- net RPI0_GPIO5: no longer J5.29 (GCLK1/GPIO5)
- net RPI0_GPIO6: no longer J5.31 (GCLK2/GPIO6)
- net UP_D+: now also U3.3 (IO2); no longer U3.1 (IO1)
- net UP_D-: now also U3.1 (IO1); no longer U3.3 (IO2)
- net VSYS: now also TP1.1
- net at C34.1, U5.3 (VBAT): now also BT1.P (+); no longer BT1.1 (+)
- net RPI0_GPIO16: no longer names the net of J7.16 (Pin_16)
- net RPI0_GPIO16: no longer J5.36 (GPIO16)
- net RPI0_GPIO22 renamed GSIN
- net GSIN: now also J4.1 (Pin_1); no longer J7.26 (Pin_26)
- net RPI0_GPIO23 renamed GSOUT
- net GSOUT: now also J4.9 (Pin_9); no longer J7.28 (Pin_28)
- net RPI0_GPIO24 renamed GCLK
- net GCLK: now also J4.2 (Pin_2); no longer J8.1 (Pin_1)
- net RPI0_GPIO25 renamed GLAT
- net GLAT: now also J4.3 (Pin_3); no longer J8.3 (Pin_3)
- net RPI0_GPIO26 renamed GSBLK
- net GSBLK: now also J4.4 (Pin_4); no longer J8.4 (Pin_4)
- net RPI0_GPIO27 renamed CLK
- net CLK: now also J4.6 (Pin_6); no longer J8.2 (Pin_2)
- new net BLK: J4.8 (Pin_8), J5.36 (GPIO16)
- new net LAT: J4.7 (Pin_7), J5.7 (GCLK0/GPIO4)
- new net SIN: J4.5 (Pin_5), J5.31 (GCLK2/GPIO6)
- new net SOUT: J4.10 (Pin_10), J5.29 (GCLK1/GPIO5)

Commit message: 3V3 + Charging + Fuel gauge PCB done
Connections:
- net 3V3: now also C57.1, U9.2 (CELL), U9.3 (VDD)
- net B+: no longer C57.1, U9.2 (CELL), U9.3 (VDD)
- net GND: now also C40.1, C41.1, C43.2, C44.2, U7.1 (GND), U8.1 (GND)
Other:
- moved on the sheet: C57
Changed lines of the file:
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@@
 	)
 	(junction
+		(at 483.87 76.2)
+		(diameter 0)
+		(color 0 0 0 0)
+	)
+	(junction
 		(at 146.05 24.13)
 		(diameter 0)
@@
 	)
 	(junction
+		(at 483.87 43.18)
+		(diameter 0)
+		(color 0 0 0 0)
+	)
+	(junction
 		(at 539.115 66.04)
 		(diameter 0)
@@
 	(wire
 		(pts
+			(xy 483.87 76.2) (xy 499.11 76.2)
+		)
+		(stroke
+			(width 0)
+			(type default)
+		)
+	)
+	(wire
+		(pts
 			(xy 559.435 41.275) (xy 559.435 42.545)
 		)
@@
 	(wire
 		(pts
-			(xy 546.1 267.335) (xy 546.1 270.51)
+			(xy 546.1 267.97) (xy 546.1 270.51)
 		)
 		(stroke
@@
 	(wire
 		(pts
-			(xy 476.885 43.18) (xy 499.11 43.18)
+			(xy 476.885 43.18) (xy 483.87 43.18)
 		)
 		(stroke
@@
 	(wire
 		(pts
-			(xy 546.1 259.715) (xy 546.1 259.08)
+			(xy 546.1 260.35) (xy 546.1 259.08)
+		)
+		(stroke
+			(width 0)
+			(type default)
+		)
+	)
+	(wire
+		(pts
+			(xy 483.87 43.18) (xy 499.11 43.18)
 		)
 		(stroke
@@
 	(wire
 		(pts
-			(xy 476.885 76.2) (xy 499.11 76.2)
+			(xy 476.885 76.2) (xy 483.87 76.2)
 		)
 		(stroke
@@
 		)
 	)
-	(global_label "B+"
+	(global_label "3V3"
 		(shape input)
 		(at 546.1 254 90)
@@
 		)
 		(property "Intersheetrefs" "${INTERSHEET_REFS}"
-			(at 546.1 248.1724 90)
+			(at 546.1 247.5072 90)
 			(effects
 				(font
@@
 	)
 	(symbol
+		(lib_name "GND_19")
+		(lib_id "power:GND")
+		(at 483.87 76.2 0)
+		(unit 1)
+		(exclude_from_sim no)
+		(in_bom yes)
+		(on_board yes)
+		(dnp no)
+		(fields_autoplaced yes)
+		(property "Reference" "#PWR064"
+			(at 483.87 82.55 0)
+			(effects
+				(font
+					(size 1.27 1.27)
+				)
+				(hide yes)
+			)
+		)
+		(property "Value" "GND"
+			(at 483.87 81.28 0)
+			(effects
+				(font
+					(size 1.27 1.27)
+				)
+			)
+		)
+		(property "Footprint" ""
+			(at 483.87 76.2 0)
+			(effects
+				(font
+					(size 1.27 1.27)
+				)
+				(hide yes)
+			)
+		)
+		(property "Datasheet" ""
+			(at 483.87 76.2 0)
+			(effects
+				(font
+					(size 1.27 1.27)
+				)
+				(hide yes)
+			)
+		)
+		(property "Description" "Power symbol creates a global label with name \"GND\" , ground"
+			(at 483.87 76.2 0)
+			(effects
+				(font
+					(size 1.27 1.27)
+				)
+				(hide yes)
+			)
+		)
+		(pin "1"
+		)
+		(instances
+			(project "vfd-tool"
+				(path "/849d9919-4175-4212-8785-6cd0421cfa2d"
+					(reference "#PWR064")
+					(unit 1)
+				)
+			)
+		)
+	)
+	(symbol
 		(lib_id "Regulator_Switching:TPS562200")
 		(at 499.11 68.58 0)
@@
 	(symbol
 		(lib_id "Device:C")
-		(at 546.1 263.525 0)
+		(at 546.1 264.16 0)
 		(unit 1)
 		(exclude_from_sim no)
@@
 		(fields_autoplaced yes)
 		(property "Reference" "C57"
-			(at 549.275 262.255 0)
+			(at 549.275 262.89 0)
 			(effects
 				(font
@@
 		)
 		(property "Value" "0.1uF"
-			(at 549.275 264.795 0)
+			(at 549.275 265.43 0)
 			(effects
 				(font
@@
 		)
 		(property "Footprint" "Capacitor_SMD:C_0402_1005Metric_Pad0.74x0.62mm_HandSolder"
-			(at 547.0652 267.335 0)
+			(at 547.0652 267.97 0)
 			(effects
 				(font
@@
 		)
 		(property "Datasheet" "~"
-			(at 546.1 263.525 0)
+			(at 546.1 264.16 0)
 			(effects
 				(font
@@
 		)
 		(property "Description" ""
-			(at 546.1 263.525 0)
+			(at 546.1 264.16 0)
 			(effects
 				(font
@@
 					(unit 1)
 				)
+			)
+		)
+	)
+	(symbol
+		(lib_name "GND_19")
+		(lib_id "power:GND")
+		(at 483.87 43.18 0)
+		(unit 1)
+		(exclude_from_sim no)
+		(in_bom yes)
+		(on_board yes)
+		(dnp no)
+		(fields_autoplaced yes)
+		(property "Reference" "#PWR063"
+			(at 483.87 49.53 0)
+			(effects
+				(font
+					(size 1.27 1.27)
+				)
+				(hide yes)
+			)
+		)
+		(property "Value" "GND"
+			(at 483.87 48.26 0)
+			(effects
+				(font
+					(size 1.27 1.27)
+				)
+			)
+		)
+		(property "Footprint" ""
+			(at 483.87 43.18 0)
+			(effects
+				(font
+					(size 1.27 1.27)
+				)
+				(hide yes)
+			)
+		)
+		(property "Datasheet" ""
+			(at 483.87 43.18 0)
+			(effects
+				(font
+					(size 1.27 1.27)
+				)
+				(hide yes)
+			)
+		)
+		(property "Description" "Power symbol creates a global label with name \"GND\" , ground"
+			(at 483.87 43.18 0)
+			(effects
+				(font
+					(size 1.27 1.27)
+				)
+				(hide yes)
+			)
+		)
+		(pin "1"
+		)
+		(instances
+			(project "vfd-tool"
+				(path "/849d9919-4175-4212-8785-6cd0421cfa2d"
+					(reference "#PWR063")
+					(unit 1)
+				)

Commit message: 5V & USB hub done
Parts:
- added C62: 0.1uF, Capacitor_SMD:C_0402_1005Metric_Pad0.74x0.62mm_HandSolder, symbol Device:C
Connections:
- net 3V3: now also C62.1
- net EXTRA_USB4_D-: no longer U2.6 (DM3)
- net GND: now also C62.2
- new net EXTRA_USB3_D-: U2.6 (DM3)
Changed lines of the file:
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@@
 	)
 	(junction
+		(at 13.97 292.1)
+		(diameter 0)
+		(color 0 0 0 0)
+	)
+	(junction
 		(at 34.29 299.72)
 		(diameter 0)
@@
 	)
 	(junction
+		(at 24.13 299.72)
+		(diameter 0)
+		(color 0 0 0 0)
+	)
+	(junction
 		(at 234.315 100.33)
 		(diameter 0)
@@
 	)
 	(junction
+		(at 24.13 292.1)
+		(diameter 0)
+		(color 0 0 0 0)
+	)
+	(junction
 		(at 546.1 259.08)
 		(diameter 0)
@@
 	(wire
 		(pts
-			(xy 24.13 292.1) (xy 34.29 292.1)
-		)
-		(stroke
-			(width 0)
-			(type default)
-		)
-	)
-	(wire
-		(pts
 			(xy 34.29 93.98) (xy 34.29 95.25)
 		)
@@
 	(wire
 		(pts
+			(xy 24.13 292.1) (xy 34.29 292.1)
+		)
+		(stroke
+			(width 0)
+			(type default)
+		)
+	)
+	(wire
+		(pts
 			(xy 64.77 292.1) (xy 73.66 292.1)
 		)
@@
 	(wire
 		(pts
+			(xy 13.97 299.72) (xy 24.13 299.72)
+		)
+		(stroke
+			(width 0)
+			(type default)
+		)
+	)
+	(wire
+		(pts
 			(xy 502.92 114.3) (xy 506.73 114.3)
 		)
@@
 	(wire
 		(pts
+			(xy 7.62 292.1) (xy 13.97 292.1)
+		)
+		(stroke
+			(width 0)
+			(type default)
+		)
+	)
+	(wire
+		(pts
 			(xy 328.93 306.07) (xy 328.93 307.34)
 		)
@@
 	(wire
 		(pts
+			(xy 13.97 292.1) (xy 24.13 292.1)
+		)
+		(stroke
+			(width 0)
+			(type default)
+		)
+	)
+	(wire
+		(pts
 			(xy 54.61 234.95) (xy 68.58 234.95)
 		)
@@
 	)
 	(rectangle
-		(start 13.97 193.04)
-		(end 264.16 349.25)
+		(start -236.22 349.25)
+		(end 13.97 193.04)
 		(stroke
 			(width 0)
@@
 	(global_label "3V3"
 		(shape input)
-		(at 24.13 292.1 180)
+		(at 7.62 292.1 180)
 		(fields_autoplaced yes)
 		(effects
@@
 		)
 		(property "Intersheetrefs" "${INTERSHEET_REFS}"
-			(at 17.6372 292.1 0)
+			(at 1.1272 292.1 0)
 			(effects
 				(font
@@
 		)
 	)
-	(global_label "EXTRA_USB4_D-"
+	(global_label "EXTRA_USB3_D-"
 		(shape input)
 		(at 127 254 0)
@@
 					(unit 1)
 				)
+			)
+		)
+	)
+	(symbol
+		(lib_id "Device:C")
+		(at 13.97 295.91 0)
+		(unit 1)
+		(exclude_from_sim no)
+		(in_bom yes)
+		(on_board yes)
+		(dnp no)
+		(property "Reference" "C62"
+			(at 16.51 295.275 0)
+			(effects
+				(font
+					(size 1.27 1.27)
+				)
+				(justify left)
+			)
+		)
+		(property "Value" "0.1uF"
+			(at 16.51 297.18 0)
+			(effects
+				(font
+					(size 1.27 1.27)
+				)
+				(justify left)
+			)
+		)
+		(property "Footprint" "Capacitor_SMD:C_0402_1005Metric_Pad0.74x0.62mm_HandSolder"
+			(at 14.9352 299.72 0)
+			(effects
+				(font
+					(size 1.27 1.27)
+				)
+				(hide yes)
+			)
+		)
+		(property "Datasheet" "~"
+			(at 13.97 295.91 0)
+			(effects
+				(font
+					(size 1.27 1.27)
+				)
+				(hide yes)
+			)
+		)
+		(property "Description" ""
+			(at 13.97 295.91 0)
+			(effects
+				(font
+					(size 1.27 1.27)
+				)
+				(hide yes)
+			)
+		)
+		(pin "1"
+		)
+		(pin "2"
+		)
+		(instances
+			(project "vfd-tool"
+				(path "/849d9919-4175-4212-8785-6cd0421cfa2d"
+					(reference "C62")
+					(unit 1)
+				)

Commit message: Flash done and the majority of the RP2040 mcu done
Connections:
- net 2040_D-: now reaches R6.1, U1.46 (USB_DM)
- net 2040_D+: now reaches R5.2, U1.47 (USB_DP)
Other:
- moved on the sheet: R5, R6
Changed lines of the file:
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@@
 	(wire
 		(pts
-			(xy 34.29 58.42) (xy 36.83 58.42)
+			(xy 27.94 58.42) (xy 30.48 58.42)
 		)
 		(stroke
@@
 	(wire
 		(pts
-			(xy 34.29 55.88) (xy 36.83 55.88)
+			(xy 27.94 55.88) (xy 30.48 55.88)
 		)
 		(stroke
@@
 	(wire
 		(pts
-			(xy 44.45 58.42) (xy 48.26 58.42)
+			(xy 38.1 58.42) (xy 48.26 58.42)
 		)
 		(stroke
@@
 	(wire
 		(pts
-			(xy 44.45 55.88) (xy 48.26 55.88)
+			(xy 38.1 55.88) (xy 48.26 55.88)
 		)
 		(stroke
@@
 	)
 	(rectangle
-		(start -236.22 349.25)
-		(end 13.97 193.04)
+		(start 13.97 193.04)
+		(end 264.16 349.25)
 		(stroke
 			(width 0)
@@
 		)
 	)
+	(label "2040_D-"
+		(at 39.37 58.42 0)
+		(fields_autoplaced yes)
+		(effects
+			(font
+				(size 1.27 1.27)
+			)
+			(justify left bottom)
+		)
+	)
+	(label "2040_D+"
+		(at 39.37 55.88 0)
+		(fields_autoplaced yes)
+		(effects
+			(font
+				(size 1.27 1.27)
+			)
+			(justify left bottom)
+		)
+	)
 	(global_label "uSD_CLK"
 		(shape input)
@@
 	(global_label "RP2040_D+"
 		(shape input)
-		(at 34.29 55.88 180)
+		(at 27.94 55.88 180)
 		(fields_autoplaced yes)
 		(effects
@@
 		)
 		(property "Intersheetrefs" "${INTERSHEET_REFS}"
-			(at 20.1168 55.88 0)
+			(at 13.7668 55.88 0)
 			(effects
 				(font
@@
 	(global_label "RP2040_D-"
 		(shape input)
-		(at 34.29 58.42 180)
+		(at 27.94 58.42 180)
 		(fields_autoplaced yes)
 		(effects
@@
 		)
 		(property "Intersheetrefs" "${INTERSHEET_REFS}"
-			(at 20.1168 58.42 0)
+			(at 13.7668 58.42 0)
 			(effects
 				(font
@@
 	(symbol
 		(lib_id "Device:R")
-		(at 40.64 58.42 270)
+		(at 34.29 58.42 270)
 		(unit 1)
 		(exclude_from_sim no)
@@
 		(dnp no)
 		(property "Reference" "R6"
-			(at 41.91 59.69 0)
+			(at 35.56 59.69 0)
 			(effects
 				(font
@@
 		)
 		(property "Value" "27.4R"
-			(at 39.37 59.69 0)
+			(at 33.02 59.69 0)
 			(effects
 				(font
@@
 		)
 		(property "Footprint" "Resistor_SMD:R_0402_1005Metric_Pad0.72x0.64mm_HandSolder"
-			(at 40.64 56.642 90)
+			(at 34.29 56.642 90)
 			(effects
 				(font
@@
 		)
 		(property "Datasheet" "~"
-			(at 40.64 58.42 0)
+			(at 34.29 58.42 0)
 			(effects
 				(font
@@
 		)
 		(property "Description" ""
-			(at 40.64 58.42 0)
+			(at 34.29 58.42 0)
 			(effects
 				(font
@@
 	(symbol
 		(lib_id "Device:R")
-		(at 40.64 55.88 90)
+		(at 34.29 55.88 90)
 		(unit 1)
 		(exclude_from_sim no)
@@
 		(dnp no)
 		(property "Reference" "R5"
-			(at 39.37 54.61 0)
+			(at 33.02 54.61 0)
 			(effects
 				(font
@@
 		)
 		(property "Value" "27.4R"
-			(at 41.91 54.61 0)
+			(at 35.56 54.61 0)
 			(effects
 				(font
@@
 		)
 		(property "Footprint" "Resistor_SMD:R_0402_1005Metric_Pad0.72x0.64mm_HandSolder"
-			(at 40.64 57.658 90)
+			(at 34.29 57.658 90)
 			(effects
 				(font
@@
 		)
 		(property "Datasheet" "~"
-			(at 40.64 55.88 0)
+			(at 34.29 55.88 0)
 			(effects
 				(font
@@
 		)
 		(property "Description" ""
-			(at 40.64 55.88 0)
+			(at 34.29 55.88 0)
 			(effects
 				(font

Commit message: 5V power done and general layour of of the PCB
Parts:
- added C63: 0.1uF, Capacitor_SMD:C_0402_1005Metric_Pad0.74x0.62mm_HandSolder, symbol Device:C
Connections:
- net 3V3: now also J3.4 (VDD), C63.1
- net GND: now also C30.2, C63.2
Other:
- moved on the sheet: C24, C30
Changed lines of the file:
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@@
 	)
 	(junction
-		(at 212.09 140.97)
-		(diameter 0)
-		(color 0 0 0 0)
-	)
-	(junction
 		(at 563.88 111.76)
 		(diameter 0)
@@
 	)
 	(junction
+		(at 215.9 134.62)
+		(diameter 0)
+		(color 0 0 0 0)
+	)
+	(junction
 		(at 392.43 307.34)
 		(diameter 0)
@@
 	)
 	(junction
+		(at 209.55 140.97)
+		(diameter 0)
+		(color 0 0 0 0)
+	)
+	(junction
 		(at 559.435 42.545)
 		(diameter 0)
@@
 	)
 	(junction
+		(at 156.21 31.75)
+		(diameter 0)
+		(color 0 0 0 0)
+	)
+	(junction
 		(at 44.45 292.1)
 		(diameter 0)
@@
 	)
 	(junction
+		(at 156.21 24.13)
+		(diameter 0)
+		(color 0 0 0 0)
+	)
+	(junction
 		(at 559.435 75.565)
 		(diameter 0)
@@
 	)
 	(junction
-		(at 157.48 24.13)
+		(at 163.83 24.13)
 		(diameter 0)
 		(color 0 0 0 0)
@@
 	(wire
 		(pts
+			(xy 156.21 31.75) (xy 163.83 31.75)
+		)
+		(stroke
+			(width 0)
+			(type default)
+		)
+	)
+	(wire
+		(pts
 			(xy 73.66 284.48) (xy 73.66 289.56)
 		)
@@
 	(wire
 		(pts
-			(xy 212.09 140.97) (xy 212.09 142.875)
+			(xy 215.9 134.62) (xy 215.9 135.89)
 		)
 		(stroke
@@
 	(wire
 		(pts
+			(xy 156.21 24.13) (xy 163.83 24.13)
+		)
+		(stroke
+			(width 0)
+			(type default)
+		)
+	)
+	(wire
+		(pts
 			(xy 511.81 220.98) (xy 514.35 220.98)
 		)
@@
 	(wire
 		(pts
+			(xy 209.55 134.62) (xy 215.9 134.62)
+		)
+		(stroke
+			(width 0)
+			(type default)
+		)
+	)
+	(wire
+		(pts
 			(xy 187.96 156.21) (xy 212.725 156.21)
 		)
@@
 	(wire
 		(pts
-			(xy 146.05 31.75) (xy 157.48 31.75)
+			(xy 146.05 31.75) (xy 156.21 31.75)
 		)
 		(stroke
@@
 	(wire
 		(pts
+			(xy 212.725 161.29) (xy 209.55 161.29)
+		)
+		(stroke
+			(width 0)
+			(type default)
+		)
+	)
+	(wire
+		(pts
 			(xy 490.22 276.225) (xy 490.22 284.48)
 		)
@@
 	(wire
 		(pts
-			(xy 213.36 140.97) (xy 212.09 140.97)
+			(xy 223.52 134.62) (xy 215.9 134.62)
 		)
 		(stroke
@@
 	(wire
 		(pts
-			(xy 146.05 24.13) (xy 157.48 24.13)
+			(xy 146.05 24.13) (xy 156.21 24.13)
 		)
 		(stroke
@@
 	(wire
 		(pts
+			(xy 209.55 161.29) (xy 209.55 140.97)
+		)
+		(stroke
+			(width 0)
+			(type default)
+		)
+	)
+	(wire
+		(pts
 			(xy 213.36 31.75) (xy 213.36 33.02)
 		)
@@
 	(wire
 		(pts
-			(xy 212.09 161.29) (xy 212.725 161.29)
+			(xy 209.55 134.62) (xy 209.55 140.97)
 		)
 		(stroke
@@
 	(wire
 		(pts
-			(xy 212.09 150.495) (xy 212.09 161.29)
-		)
-		(stroke
-			(width 0)
-			(type default)
-		)
-	)
-	(wire
-		(pts
-			(xy 157.48 24.13) (xy 159.385 24.13)
+			(xy 163.83 24.13) (xy 165.735 24.13)
 		)
 		(stroke
@@
 	(wire
 		(pts
-			(xy 203.2 140.97) (xy 212.09 140.97)
+			(xy 203.2 140.97) (xy 209.55 140.97)
 		)
 		(stroke
@@
 	(global_label "3V3"
 		(shape input)
-		(at 159.385 24.13 0)
+		(at 165.735 24.13 0)
 		(fields_autoplaced yes)
 		(effects
@@
 		)
 		(property "Intersheetrefs" "${INTERSHEET_REFS}"
-			(at 165.7984 24.13 0)
+			(at 172.1484 24.13 0)
 			(effects
 				(font
@@
 	(global_label "3V3"
 		(shape input)
-		(at 213.36 140.97 0)
+		(at 223.52 134.62 0)
 		(fields_autoplaced yes)
 		(effects
@@
 		)
 		(property "Intersheetrefs" "${INTERSHEET_REFS}"
-			(at 219.7734 140.97 0)
+			(at 229.9334 134.62 0)
 			(effects
 				(font
@@
 	)
 	(symbol
+		(lib_id "Device:C")
+		(at 156.21 27.94 0)
+		(unit 1)
+		(exclude_from_sim no)
+		(in_bom yes)
+		(on_board yes)
+		(dnp no)
+		(property "Reference" "C63"
+			(at 158.75 27.305 0)
+			(effects
+				(font
+					(size 1.27 1.27)
+				)
+				(justify left)
+			)
+		)
+		(property "Value" "0.1uF"
+			(at 158.75 29.21 0)
+			(effects
+				(font
+					(size 1.27 1.27)
+				)
+				(justify left)
+			)
+		)
+		(property "Footprint" "Capacitor_SMD:C_0402_1005Metric_Pad0.74x0.62mm_HandSolder"
+			(at 157.1752 31.75 0)
+			(effects
+				(font
+					(size 1.27 1.27)
+				)
+				(hide yes)
+			)
+		)
+		(property "Datasheet" "~"
+			(at 156.21 27.94 0)
+			(effects
+				(font
+					(size 1.27 1.27)
+				)
+				(hide yes)
+			)
+		)
+		(property "Description" ""
+			(at 156.21 27.94 0)
+			(effects
+				(font
+					(size 1.27 1.27)
+				)
+				(hide yes)
+			)
+		)
+		(pin "1"
+		)
+		(pin "2"
+		)
+		(instances
+			(project "vfd-tool"
+				(path "/849d9919-4175-4212-8785-6cd0421cfa2d"
+					(reference "C63")
+					(unit 1)
+				)
+			)
+		)
+	)
+	(symbol
 		(lib_id "Device:R_Small")
 		(at 455.93 201.93 0)
@@
 	(symbol
 		(lib_id "Device:C")
-		(at 212.09 146.685 0)
+		(at 215.9 139.7 0)
 		(unit 1)
 		(exclude_from_sim no)
@@
 		(dnp no)
 		(property "Reference" "C30"
-			(at 215.9 145.415 0)
+			(at 219.71 138.43 0)
 			(effects
 				(font
@@
 		)
 		(property "Value" "10uF"
-			(at 220.345 145.415 0)
+			(at 224.155 138.43 0)
 			(effects
 				(font
@@
 		)
 		(property "Footprint" "Capacitor_SMD:C_0603_1608Metric"
-			(at 213.0552 150.495 0)
+			(at 216.8652 143.51 0)
 			(effects
 				(font
@@
 		)
 		(property "Datasheet" "~"
-			(at 212.09 146.685 0)
+			(at 215.9 139.7 0)
 			(effects
 				(font
@@
 		)
 		(property "Description" ""
-			(at 212.09 146.685 0)
+			(at 215.9 139.7 0)
 			(effects
 				(font
@@
 	)
 	(symbol
+		(lib_id "power:GND")
+		(at 215.9 143.51 0)
+		(unit 1)
+		(exclude_from_sim no)
+		(in_bom yes)
+		(on_board yes)
+		(dnp no)
+		(property "Reference" "#PWR065"
+			(at 215.9 149.86 0)
+			(effects
+				(font
+					(size 1.27 1.27)
+				)
+				(hide yes)
+			)
+		)
+		(property "Value" "GND"
+			(at 219.964 145.542 0)
+			(effects
+				(font
+					(size 1.27 1.27)
+				)
+			)
+		)
+		(property "Footprint" ""
+			(at 215.9 143.51 0)
+			(effects
+				(font
+					(size 1.27 1.27)
+				)
+				(hide yes)
+			)
+		)
+		(property "Datasheet" ""
+			(at 215.9 143.51 0)
+			(effects
+				(font
+					(size 1.27 1.27)
+				)
+				(hide yes)
+			)
+		)
+		(property "Description" ""
+			(at 215.9 143.51 0)
+			(effects
+				(font
+					(size 1.27 1.27)
+				)
+				(hide yes)
+			)
+		)
+		(pin "1"
+		)
+		(instances
+			(project "vfd-tool"
+				(path "/849d9919-4175-4212-8785-6cd0421cfa2d"
+					(reference "#PWR065")
+					(unit 1)
+				)
+			)
+		)
+	)
+	(symbol
 		(lib_id "Device:C")
 		(at 551.815 69.85 180)
@@
 	(symbol
 		(lib_id "Device:C")
-		(at 157.48 27.94 0)
+		(at 163.83 27.94 0)
 		(unit 1)
 		(exclude_from_sim no)
@@
 		(dnp no)
 		(property "Reference" "C24"
-			(at 160.02 27.305 0)
+			(at 166.37 27.305 0)
 			(effects
 				(font
@@
 		)
 		(property "Value" "0.1uF"
-			(at 160.02 29.21 0)
+			(at 166.37 29.21 0)
 			(effects
 				(font
@@
 		)
 		(property "Footprint" "Capacitor_SMD:C_0402_1005Metric_Pad0.74x0.62mm_HandSolder"
-			(at 158.4452 31.75 0)
+			(at 164.7952 31.75 0)
 			(effects
 				(font
@@
 		)
 		(property "Datasheet" "~"
-			(at 157.48 27.94 0)
+			(at 163.83 27.94 0)
 			(effects
 				(font
@@
 		)
 		(property "Description" ""
-			(at 157.48 27.94 0)
+			(at 163.83 27.94 0)
 			(effects
 				(font

Commit message: finished interconnect, started on internal power layer
Parts:
- TP3, TP4: footprint TestPoint:TestPoint_Pad_D3.0mm -> TestPoint:TestPoint_Pad_D1.0mm
Connections:
- net GPIO16 is gone; now on net BATT_INT: U9.5 (~{ALERT})
- net 3V3: now also J6.7 (Pin_7), J6.9 (Pin_9); no longer J6.15 (Pin_15), J6.17 (Pin_17)
- net 5V: now also J6.11 (Pin_11), J6.13 (Pin_13); no longer J6.19 (Pin_19), J6.21 (Pin_21)
- net EXTRA_USB3_D-: now also J6.26 (Pin_26)
- net EXTRA_USB4_D-: no longer J6.26 (Pin_26)
- net GND: now also J6.15 (Pin_15); no longer J6.13 (Pin_13), J8.10 (Pin_10)
- net RP2040_GPIO27: no longer J8.12 (Pin_12)
- net RP2040_GPIO28: no longer J8.14 (Pin_14)
- net VBUS: now also J6.17 (Pin_17), J6.19 (Pin_19), J6.21 (Pin_21); no longer J6.11 (Pin_11), J6.7 (Pin_7), J6.9 (Pin_9)
